Commit message: FIX : camera description

File: carrier_ros_description/urdf/_d435.urdf.xacro (robot description, xacro)
@@ -10,5 +10,5 @@
   <xacro:include filename="$(find carrier_ros_description)/urdf/_materials.urdf.xacro" />
   <xacro:include filename="$(find carrier_ros_description)/urdf/_usb_plug.urdf.xacro" />
-  <xacro:macro name="sensor_d435" params="parent *origin name:=camera use_nominal_extrinsics:=false add_plug:=false use_mesh:=true">
+  <xacro:macro name="sensor_d435" params="parent *origin name:=camera use_nominal_extrinsics:=true add_plug:=false use_mesh:=true">
     <xacro:property name="M_PI" value="3.1415926535897931" />
     <!-- The following values are approximate, and the camera node

File: carrier_ros_description/urdf/carrier_ros.urdf.g2.xacro (robot description, xacro)
@@ -3,5 +3,5 @@
   <xacro:include filename="$(find carrier_ros_description)/urdf/common_properties.xacro"/>
   <xacro:include filename="$(find carrier_ros_description)/urdf/_d435.urdf.xacro" />
-  <xacro:arg name="use_nominal_extrinsics" default="false"/>
+  <xacro:arg name="use_nominal_extrinsics" default="true"/>
   <xacro:arg name="add_plug" default="false" />
   <xacro:arg name="use_mesh" default="true" />
